File: Hardware/teensy3.5dds.brd (EAGLE design)
At the start: 110 x 85 mm, 96 parts, among them IC1 AD8034, IC2 AD8034, IC3 AD8034, IC5 AD8034, IC6 AD737KRZ-R7, IC7 AD8034, IC8 AD8034, J1 1776275-2, J2 1776275-2, Q1 10MHz, U1 TEENSY_3.5/3.6_BASIC, U2 ATMEGA32U4-AU, X1 1-227161-0

Commit message: board redisegn
Parts:
- removed C11: (no value), rcl:C0805
- removed C12: 100n, rcl:C0805
- added U$3, U$4, U$5: (no value), holes:3,0
- moved R15 173.5 mm to (91.9, 95.4), turned to 180 degrees
- moved C25 173.4 mm to (90.9, 91.8), turned to 90 degrees
- moved R8 140.3 mm to (81.3, 95.4), turned to 180 degrees
- moved R4 139.5 mm to (89.4, 82.4)
- moved R7 138.7 mm to (89.4, 84.8)
- moved R10 135.4 mm to (86.6, 95.4), turned to 180 degrees
- moved IC2 134.3 mm to (83.9, 89.2), turned to 270 degrees
- moved R13 119.9 mm to (84.5, 80.0), turned to 180 degrees
- moved J2 105.2 mm to (5.09, 58.4)
- moved J1 100.5 mm to (5.08, 70.6)
- moved R42 74.0 mm to (5.71, 37.1), turned to 270 degrees
- moved R41 68.9 mm to (1.52, 37.1), turned to 270 degrees
- moved R43 68.8 mm to (3.30, 28.2)
- moved S1 42.8 mm to (11.6, 20.4), turned to 270 degrees
- moved R35 26.3 mm to (91.2, 64.8)
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Connections:
- net GND: no longer C11.2, C12.1
- net N$25: now also U2.32; no longer U2.30
- net N$29: now also U2.30; no longer U2.29
- net N$8: now also U2.31; no longer U2.12
- net V+: no longer C11.1
- net V-: no longer C12.2
Routing:
- net GND: track 826.6 -> 0.00 mm, vias 18 -> 0
- net +5V: track 295.6 -> 71.3 mm, vias 1 -> 4
- net N$25: track 0.00 -> 68.7 mm, vias 0 -> 2
- net N$8: track 0.00 -> 68.1 mm, vias 0 -> 2
- net N$29: track 0.00 -> 62.9 mm, vias 0 -> 1
- net N$19: track 71.3 -> 40.6 mm
- net N$34: track 0.00 -> 30.7 mm
- net N$3: track 91.7 -> 64.6 mm
- net N$62: track 45.5 -> 18.5 mm
- net V-: track 91.4 -> 68.7 mm, vias 9 -> 7
- net N$2: track 34.2 -> 16.5 mm
- net DAC0_FILTERED: track 40.9 -> 24.2 mm
- net N$1: track 0.00 -> 16.1 mm
- net N$28: track 0.00 -> 13.4 mm
- net N$27: track 0.00 -> 12.7 mm
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- added copper zone on layer 16, net +5V
- added copper zone on layer 1, net GND
- added copper zone on layer 16, net GND
- removed copper zone on layer 1, net V+
- removed copper zone on layer 16, net V-
Other:
- board size 110 x 85 mm -> 95.8 x 84.1 mm
