File: Hardware/teensy3.5dds.sch (EAGLE design)
At the start: 94 parts, among them IC1 AD8034, IC2 AD8034, IC3 AD8034, IC5 AD8034, IC6 AD737KRZ-R7, IC7 AD8034, IC8 AD8034, J1 1776275-2, J2 1776275-2, Q1 10MHz, U1 TEENSY_3.5/3.6_BASIC, U2 ATMEGA32U4-AU, X1 1-227161-0

Commit message: fixes following the advice of people better than me at making PCBs
Connections:
- removed net V-1: R13.A
- net DAC0: now also IC1B.+IN; no longer IC1A.+IN
- net DAC0_OFFSET: now also IC1A.OUT; no longer IC1B.OUT
- net N$21: now also IC1A.-IN; no longer IC1B.-IN
- net N$23: now also IC1B.-IN, IC1B.OUT; no longer IC1A.-IN, IC1A.OUT
- net N$26: now also IC1A.+IN; no longer IC1B.+IN
- net V-: now also R13.A
Other:
- moved on the sheet: IC1A, IC1B
Changed lines of the file:
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@@
 <attribute name="NAME" x="335.026" y="-77.978" size="1.778" layer="95" rot="MR0"/>
 </instance>
-<instance part="IC1" gate="A" x="64.77" y="-27.94" smashed="yes">
-<attribute name="NAME" x="62.23" y="-22.86" size="1.778" layer="95"/>
-<attribute name="VALUE" x="62.23" y="-34.29" size="1.778" layer="96"/>
-</instance>
-<instance part="IC1" gate="B" x="100.33" y="-30.48" smashed="yes">
-<attribute name="NAME" x="102.87" y="-27.305" size="1.778" layer="95"/>
-<attribute name="VALUE" x="100.33" y="-35.56" size="1.778" layer="96"/>
+<instance part="IC1" gate="A" x="100.33" y="-30.48" smashed="yes">
+<attribute name="NAME" x="97.79" y="-25.4" size="1.778" layer="95"/>
+<attribute name="VALUE" x="97.79" y="-36.83" size="1.778" layer="96"/>
+</instance>
+<instance part="IC1" gate="B" x="64.77" y="-27.94" smashed="yes">
+<attribute name="NAME" x="67.31" y="-24.765" size="1.778" layer="95"/>
+<attribute name="VALUE" x="64.77" y="-33.02" size="1.778" layer="96"/>
 </instance>
 <instance part="R9" gate="G$1" x="85.09" y="-35.56" smashed="yes" rot="R90">
@@
 </segment>
 <segment>
-<pinref part="IC1" gate="A" pin="+IN"/>
+<pinref part="IC1" gate="B" pin="+IN"/>
 <wire x1="57.15" y1="-25.4" x2="50.8" y2="-25.4" width="0.1524" layer="91"/>
 <label x="50.8" y="-25.4" size="1.778" layer="95"/>
@@
 </segment>
 <segment>
-<wire x1="77.47" y1="-48.26" x2="72.39" y2="-48.26" width="0.1524" layer="91"/>
-<pinref part="R5" gate="G$1" pin="A"/>
-</segment>
-<segment>
 <pinref part="C2" gate="G$1" pin="2"/>
 <wire x1="50.8" y1="2.54" x2="50.8" y2="0" width="0.1524" layer="91"/>
@@
 <wire x1="281.94" y1="-101.6" x2="287.02" y2="-101.6" width="0.1524" layer="91"/>
 <label x="284.48" y="-101.6" size="1.778" layer="95"/>
+</segment>
+<segment>
+<pinref part="R5" gate="G$1" pin="A"/>
+<wire x1="77.47" y1="-48.26" x2="73.66" y2="-48.26" width="0.1524" layer="91"/>
+<label x="73.66" y="-48.26" size="1.778" layer="95"/>
+</segment>
+<segment>
+<wire x1="157.48" y1="-2.54" x2="152.4" y2="-2.54" width="0.1524" layer="91"/>
+<pinref part="R13" gate="G$1" pin="A"/>
+<label x="152.4" y="-2.54" size="1.778" layer="95"/>
 </segment>
 </net>
@@
 </segment>
 <segment>
-<pinref part="IC1" gate="B" pin="OUT"/>
-<wire x1="110.49" y1="-30.48" x2="107.95" y2="-30.48" width="0.1524" layer="91"/>
 <label x="113.03" y="-30.48" size="1.778" layer="95"/>
 <pinref part="R14" gate="G$1" pin="1"/>
-<wire x1="135.89" y1="-30.48" x2="110.49" y2="-30.48" width="0.1524" layer="91"/>
-<junction x="110.49" y="-30.48"/>
+<wire x1="135.89" y1="-30.48" x2="111.76" y2="-30.48" width="0.1524" layer="91"/>
 <pinref part="R12" gate="G$1" pin="1"/>
+<wire x1="111.76" y1="-30.48" x2="110.49" y2="-30.48" width="0.1524" layer="91"/>
 <wire x1="105.41" y1="-38.1" x2="110.49" y2="-38.1" width="0.1524" layer="91"/>
 <wire x1="110.49" y1="-38.1" x2="110.49" y2="-30.48" width="0.1524" layer="91"/>
+<pinref part="IC1" gate="A" pin="OUT"/>
+<wire x1="110.49" y1="-30.48" x2="107.95" y2="-30.48" width="0.1524" layer="91"/>
 </segment>
 </net>
@@
 <net name="N$21" class="0">
 <segment>
-<pinref part="IC1" gate="B" pin="-IN"/>
-<wire x1="92.71" y1="-33.02" x2="90.17" y2="-33.02" width="0.1524" layer="91"/>
 <wire x1="90.17" y1="-33.02" x2="90.17" y2="-38.1" width="0.1524" layer="91"/>
 <pinref part="R12" gate="G$1" pin="2"/>
@@
 <wire x1="90.17" y1="-38.1" x2="90.17" y2="-39.37" width="0.1524" layer="91"/>
 <junction x="90.17" y="-38.1"/>
+<pinref part="IC1" gate="A" pin="-IN"/>
+<wire x1="92.71" y1="-33.02" x2="90.17" y2="-33.02" width="0.1524" layer="91"/>
 </segment>
 </net>
 <net name="N$23" class="1">
 <segment>
-<pinref part="IC1" gate="A" pin="OUT"/>
+<wire x1="53.34" y1="-30.48" x2="53.34" y2="-34.29" width="0.1524" layer="91"/>
+<wire x1="53.34" y1="-34.29" x2="73.66" y2="-34.29" width="0.1524" layer="91"/>
+<pinref part="IC1" gate="B" pin="-IN"/>
+<wire x1="53.34" y1="-30.48" x2="57.15" y2="-30.48" width="0.1524" layer="91"/>
 <pinref part="R11" gate="G$1" pin="1"/>
-<wire x1="73.66" y1="-27.94" x2="72.39" y2="-27.94" width="0.1524" layer="91"/>
-<pinref part="IC1" gate="A" pin="-IN"/>
-<wire x1="57.15" y1="-30.48" x2="53.34" y2="-30.48" width="0.1524" layer="91"/>
-<wire x1="53.34" y1="-30.48" x2="53.34" y2="-34.29" width="0.1524" layer="91"/>
-<wire x1="53.34" y1="-34.29" x2="72.39" y2="-34.29" width="0.1524" layer="91"/>
-<wire x1="72.39" y1="-34.29" x2="72.39" y2="-27.94" width="0.1524" layer="91"/>
-<junction x="72.39" y="-27.94"/>
+<wire x1="73.66" y1="-27.94" x2="73.66" y2="-34.29" width="0.1524" layer="91"/>
+<pinref part="IC1" gate="B" pin="OUT"/>
+<wire x1="72.39" y1="-27.94" x2="73.66" y2="-27.94" width="0.1524" layer="91"/>
+<junction x="73.66" y="-27.94"/>
 </segment>
 </net>
@@
 <segment>
 <pinref part="R11" gate="G$1" pin="2"/>
-<pinref part="IC1" gate="B" pin="+IN"/>
 <wire x1="83.82" y1="-27.94" x2="85.09" y2="-27.94" width="0.1524" layer="91"/>
 <pinref part="R9" gate="G$1" pin="2"/>
-<wire x1="85.09" y1="-27.94" x2="92.71" y2="-27.94" width="0.1524" layer="91"/>
 <wire x1="85.09" y1="-30.48" x2="85.09" y2="-27.94" width="0.1524" layer="91"/>
+<pinref part="IC1" gate="A" pin="+IN"/>
+<wire x1="92.71" y1="-27.94" x2="85.09" y2="-27.94" width="0.1524" layer="91"/>
 <junction x="85.09" y="-27.94"/>
 </segment>
 </net>
-<net name="V-1" class="2">
-<segment>
-<wire x1="157.48" y1="-2.54" x2="152.4" y2="-2.54" width="0.1524" layer="91"/>
-<pinref part="R13" gate="G$1" pin="A"/>
-</segment>
-</net>

Commit message: board v1.0
Parts:
- removed C30, C34: 100p, rcl:C-EUC0805
- removed C32: 10p, rcl:C-EUC0805
- removed IC8: AD8034, linear:TL082D
- removed R43: (no value), rcl:R-EU_R0805
- added C11, C12: 100n, rcl:C-EUC0805
- added C26: 100p, rcl:C-EUC0805
- added IC4: AD8034, linear:TL082D
- added R19: 1k, rcl:R-EU_R0805
- added R21: 787, rcl:R-EU_M0805
- added R23: 10k, Potentiometer_vertical:POTENTIOMETER_VERTICAL
- C1: value 100n -> 1u; device rcl:C-EUC0805 -> rcl:C-EUC1206
- C19: device rcl:C-EUC1206 -> rcl:C-EUC0805
- C22: value 100n -> 10p
- C23: value 1u -> 150p
- C25: value (none) -> 1p
- C27: value 100p -> 10p
- C28: value 10p -> 100p
- C3: value 1u -> 22p; device rcl:C-EUC1206 -> rcl:C-EUC0805
- C4: value 100n -> 22p
- C5: device rcl:C-EUC0805 -> rcl:C-EUC1206
- C7: value 22p -> 1u
- C8: value 22p -> 100n
- IC5: value AD8034 -> AD737KRZ-R7; device linear:TL082D -> AD737KRZ-R7:AD737KRZ-R7
- IC6: value AD737KRZ-R7 -> AD8034; device AD737KRZ-R7:AD737KRZ-R7 -> linear:TL082D
- Q1: value 10MHz -> 16MHz
- R12: value 1k -> 500; device rcl:R-EU_R0805 -> rcl:R-EU_M0805
- R13: value 100k -> 500; device rcl:R-TRIMM3296W -> rcl:R-EU_M0805
- R15: value (none) -> 2.74k
- R16: value (none) -> 100k; device rcl:R-EU_M0805 -> rcl:R-TRIMM3296W
- R17: value (none) -> 1k; device rcl:R-EU_M0805 -> rcl:R-EU_R0805
- R18: value 2.74k -> 1k
- R20: value 787 -> 1k; device rcl:R-EU_M0805 -> rcl:R-EU_R0805
- R22: value 14.3k -> 1k; device rcl:R-EU_M0805 -> rcl:R-EU_R0805
- R25: value 10k -> 1.5k; device Potentiometer_vertical:POTENTIOMETER_VERTICAL -> rcl:R-EU_R0805
- R26: value (none) -> 14.3k; device rcl:R-EU_R0805 -> rcl:R-EU_M0805
- R27, R42: value (none) -> 50
- R28, R37: value (none) -> 5k
- R30, R41: value (none) -> 1k
- R31: value 10k -> 2k; device Potentiometer_vertical:POTENTIOMETER_VERTICAL -> rcl:R-EU_M0805
- R32: value 562 -> 10k; device rcl:R-EU_R0805 -> Potentiometer_vertical:POTENTIOMETER_VERTICAL
- R33: value 243 -> 10k
- R34: value 20k -> 562
- R35: value 1.78k -> (none); device rcl:R-EU_M0805 -> rcl:R-EU_R0805
- R36: value (none) -> 20k
- R38: value (none) -> 10k
- R39: value (none) -> 14.3k
- R4, R9: value 1k -> 10k
- R40: value 50 -> (none)
- R5: value 100k -> 10k; device rcl:R-TRIMM3296W -> rcl:R-EU_R0805
- R6: value 1k -> 100k; device rcl:R-EU_R0805 -> rcl:R-TRIMM3296W
- RL1, RL2: value PRME_15005SOCKET -> PRME_15005NOSOCKET; device prme15005:PRME_15005SOCKET -> prme15005:PRME_15005NOSOCKET
- renumbered J_DAC0_OUT to JDAC0_OUT, J_DISPLAY to JDISPLAY, J_SPI to JSPI, J_SQUARE_OUT to JSQUARE_OUT
Connections:
- removed net N$20: R13.S, R4.1
- new net N$36: IC6A.-IN, R35.2, R40.1
- new net N$37: IC7B.-IN, R16.S, R18.1
- net +5V: now also C1.1, C2.1, C5.1, C7.1, R4.1, R5.1; no longer C19.1, C22.1, C23.1, C3.1, R41.1, R42.1
- net AMPL_MEASURE: now also IC4B.OUT, R41.2, U2.PF6(ADC6/TDO); no longer IC5B.OUT, R39.2, U2.PF5(ADC5/TMS)
- net DAC0_FILTERED: now also C28.1; no longer C34.1
- net DAC0_OFFSET: now also R11.1; no longer R12.1
- net DAC0_SEL: now also R13.1, U1.22/A8; no longer R17.1, U1.36/A17
- net GND: now also C10.2, C11.1, C12.2, C13.1, C14.2, C15.1, C16.2, C17.1, C18.2, C19.1, C2.2, C22.1, C27.1, C3.1, C4.1, C5.2, C7.2, C8.2, C9.1, IC5.COM, IC5.POWER_DOWN, IC6A.+IN, R10.2, R19.2, R9.1; no longer C10.1, C13.2, C14.1, C15.2, C16.1, C17.2, C18.1, C19.2, C2.1, C22.2, C23.2, C28.1, C3.2, C32.1, C4.2, C5.1, C7.1, C8.1, C9.2, IC6.COM, IC6.POWER_DOWN, IC7B.-IN, R43.1, R6.2, R8.2
- net INTERRUPT: now also U1.21/A7, U2.PD5(XCK/CTS); no longer U1.37/A18, U2.PD4(ICP1/ADC8)
- net N$1: now also R31.2, R33.1; no longer R33.2, R35.1
- net N$10: now also R22.1; no longer R24.1
- net N$11: now also IC4A.-IN; no longer IC5A.-IN
- net N$13: now also IC4A.+IN, R24.1, R25.2; no longer IC5A.+IN, R26.1, R27.2
- net N$14: now also IC5.OUTPUT, R37.1; no longer IC6.OUTPUT, R36.1
- net N$15: now also R32.1; no longer R31.1
- net N$16: now also IC4B.-IN, R37.2, R41.1; no longer IC5B.-IN, R36.2, R39.1
- net N$17: now also R12.2; no longer R16.2
- net N$18: now also R13.2; no longer R17.2
- net N$19: now also IC6A.OUT, R40.2, R42.1; no longer IC8A.-IN, IC8A.OUT, R40.1
- net N$21: now also R10.1, R11.2; no longer R12.2, R6.1
- net N$22: now also IC4B.+IN, R38.2, R39.1; no longer IC5B.+IN, R37.2, R38.1
- net N$23: now also R7.1; no longer R11.1
- net N$24: now also R19.1, R20.2; no longer R10.2, R8.1
- net N$25: now also R4.2, U2.PF1(ADC1); no longer R41.2, U2.PC7(ICP3/CLK0/OC4A)
- net N$26: now also R7.2, R8.2; no longer R11.2, R9.2
- net N$27: now also R17.1; no longer R7.1
- net N$28: now also R17.2, R18.2; no longer R4.2, R7.2
- net N$29: now also R9.2, U2.PF4(ADC4/TCK); no longer R43.2, U2.PB6(OC1B/OC4B/ADC13)
- net N$3: now also IC6B.+IN, R23.3; no longer IC8B.+IN, R25.3
- net N$31: now also C3.2; no longer C7.2
- net N$34: now also R27.1, R31.1; no longer R15.1, R33.1
- net N$4: now also C4.2; no longer C8.2
- net N$5: now also IC6B.-IN, R22.2; no longer IC8B.-IN, R24.2
- net N$50: now also C23.2, R15.1; no longer C27.2, R18.1
- net N$53: now also C23.1, R21.1; no longer C27.1, R20.1
- net N$56: now also R6.S, R8.1; no longer R5.S, R9.1
- net N$58: now also C22.2, R15.2; no longer C24.2, R18.2
- net N$6: now also R42.2; no longer R40.2
- net N$61: now also C26.1, R21.2, R26.1; no longer C30.1, R20.2, R22.1
- net N$62: now also C26.2, R34.1; no longer C30.2, R32.1
- net N$63: now also C24.2, R26.2; no longer C28.2, R22.2
- net N$73: now also C28.2, R34.2, R36.1; no longer C34.2, R32.2, R34.1
- net N$75: now also C27.2, R36.2; no longer C32.2, R34.2
- net N$8: now also R5.2, U2.PF0(ADC0); no longer R42.2, U2.PC6(OC3A/!OC4A)
- net N$9: now also IC5.VIN, IC6B.OUT, R32.2, R32.3, R35.1; no longer IC6.VIN, IC8A.+IN, IC8B.OUT, R31.2, R31.3
- net OFF_MEASURE: now also IC4A.OUT, U2.PF7(ADC7(TDI); no longer IC5A.OUT, U2.PF6(ADC6/TDO)
- net RX1: now also U1.1/TX; no longer U1.32/A13
- net SQUARE: now also U1.A22/DAC1; no longer U1.39/A20
- net SQUARE_FILTERED: now also R33.2; no longer R35.2
- net SQUARE_OFFSET: now also R20.1, R27.2; no longer R10.1, R15.2
- net SQUARE_SEL: now also R12.1, U1.23/A9; no longer R16.1, U1.35/A16
- net TX1: now also U1.0/RX; no longer U1.31/A12
- net V+: now also C10.1, C12.1, C14.1, C16.1, C18.1, C8.1, IC1P.V+, IC2P.V+, IC3P.V+, IC4P.V+, IC5.+VS, IC6P.V+, IC7P.V+, R16.E, R23.2, R24.2, R38.1, R6.E; no longer C1.1, C13.1, C15.1, C17.1, C4.1, C9.1, IC6.+VS, R13.E, R25.2, R26.2, R37.1, R5.E
- net V-: now also C11.2, C13.2, C15.2, C17.2, C19.2, C9.2, IC1P.V-, IC2P.V-, IC3P.V-, IC4P.V-, IC5.-VS, IC5.CAV, IC6P.V-, IC7P.V-, R16.A, R23.1, R39.2, R6.A; no longer C10.2, C14.2, C16.2, C18.2, C2.2, C5.2, IC6.-VS, IC6.CAV, R13.A, R27.1, R38.2, R5.A
Other:
- moved on the sheet: C1, C10, C13, C14, C15, C16, C17, C18, C19, C2, C20, C21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

Commit message: hardware: board v2.0
correct a few derps with missing resistors
correct encoder pushbutton
add i2c pullup resistors
move some 32u4 pins to more accessible ones, supported by the arduino micro bootloader
wire the 5v led to the builtin led on 32u4
remove the ad737, move the a non-inverting summer circuit (wave+offset) with a peak finder to get the peak of the wave no matter the offset condition
Parts:
- removed C20, C21: 100n, rcl:C-EUC0805
- removed IC5: AD737KRZ-R7, AD737KRZ-R7:AD737KRZ-R7
- added C29: (no value), rcl:C-EUC0805
- added D4: (no value), diode:DIODE-SOD123
- added R43, R44, R45, R46: (no value), rcl:R-EU_R0805
- C1: value 1u -> 100u
- C5: value 100n -> 100u
- C7: value 1u -> 100n
- R1, R12, R13, R21, R26, R31, R33: device rcl:R-EU_M0805 -> rcl:R-EU_R0805
Connections:
- removed net N$14 (its old number): IC5.OUTPUT, R37.1
- removed net N$35: R2.1, SW1.P$2, U2./RESET
- removed net SS: JSPI.2, U2.PB0(SS)
- new net N$20: D4.A, IC4B.OUT, R41.2
- new net N$22: IC6A.+IN, R46.2
- new net N$38: LED1.C, R1.2
- new net RST: JSPI.2, R2.1, SW1.P$2, U2./RESET
- net +5V: now also R44.2, R45.1, S1.E; no longer R1.2
- net AMPL_MEASURE: now also C29.1, D4.C, R43.2; no longer IC4B.OUT, R41.2
- net GND: now also C29.2, R1.1, R39.2, R43.1, R46.1; no longer C20.2, C21.1, IC5.COM, IC5.POWER_DOWN, IC6A.+IN, LED1.C, S1.E
- net INTERRUPT: now also U2.PD4(ICP1/ADC8); no longer U2.PD5(XCK/CTS)
- net MISO: now also JSPI.6; no longer JSPI.3
- net MOSI: now also JSPI.3; no longer JSPI.6
- net N$3: now also R38.1
- net N$30: now also U2.PC7(ICP3/CLK0/OC4A); no longer R1.1
- net N$9: now also R37.1; no longer IC5.VIN
- net SCL: now also R45.2
- net SDA: now also R44.1
- net V+: no longer C20.1, IC5.+VS, R38.1
- net V-: no longer C21.2, IC5.-VS, IC5.CAV, R39.2
Other:
- note added: "PLACE ONE CLOSE TO EACH OPAMP IC SUPPLY"
- note removed: "PLACE ONE CLOSE TO EACH OPAMP AND AD737 IC SUPPLY"
- moved on the sheet: C1, C10, C11, C12, C13, C14, C15, C16, C17, C18, C19, C2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
